Commit message: Working code for multiple bots
chaotic because of high computation, needs refinements in code

File: omni_bot/src/bot.xacro (robot description, xacro)
@@ -11,8 +11,29 @@
             <mesh filename="package://omni_bot/src/Wheel2_Double_ohneRaeder.stl" scale=".0021 .0021 .0021"/>
           </geometry>
-          <friction>
-            <mu>0.4</mu>
-            <mu2>0.4</mu2>
-          </friction>
+          <!--<surface>
+            <friction>
+              <ode>
+                <mu>1.5</mu>
+                <mu2>1.5</mu2>
+                <fdir1>0.000000 0.000000 0.000000</fdir1>
+                <slip1>0.000000</slip1>
+                <slip2>0.000000</slip2>
+              </ode>
+            </friction>
+            <bounce>
+              <restitution_coefficient>0.000000</restitution_coefficient>
+              <threshold>100000.000000</threshold>
+            </bounce>
+            <contact>
+              <ode>
+                <soft_cfm>0.000000</soft_cfm>
+                <soft_erp>0.200000</soft_erp>
+                <kp>100000.000000</kp>
+                <kd>1.000000</kd>
+                <max_vel>100.000000</max_vel>
+                <min_depth>0.001000</min_depth>
+              </ode>
+            </contact>
+          </surface>-->
          </collision>
       <visual>
@@ -25,13 +46,8 @@
           <origin xyz="0 0 0" rpy="${roll} ${pit} ${yaw}"/>
          <mass value = "0.55"/>
-    <inertia ixx="0.0005" ixy ="0" ixz="0" iyy="0.001" iyz="0" izz="0.001"/>
+    <inertia ixx="0.0005" ixy ="0" ixz="0" iyy="0.0005" iyz="0" izz="0.001"/>
     </inertial>
-    <gazebo>
       <gravity> 1 </gravity>
-      <dampingFactor>0.4</dampingFactor>
-      <mu1>0.4</mu1>
-      <mu2>0.4</mu2>
-      <selfCollide>1</selfCollide>
-    </gazebo>
+      <selfCollide>0</selfCollide>
       </link>
      <link name="roller1${pos}">
@@ -41,8 +57,29 @@
             <mesh filename="package://omni_bot/src/Wheel2_wheel_rightOrient.stl" scale=".0021 .0021 .0021"/>
           </geometry>
-          <friction>
-            <mu>0.4</mu>
-            <mu2>0.4</mu2>
-          </friction>
+          <!--<surface>
+            <friction>
+              <ode>
+                <mu>1.5</mu>
+                <mu2>1.5</mu2>
+                <fdir1>0.000000 0.000000 0.000000</fdir1>
+                <slip1>0.000000</slip1>
+                <slip2>0.000000</slip2>
+              </ode>
+            </friction>
+            <bounce>
+              <restitution_coefficient>0.000000</restitution_coefficient>
+              <threshold>100000.000000</threshold>
+            </bounce>
+            <contact>
+              <ode>
+                <soft_cfm>0.000000</soft_cfm>
+                <soft_erp>0.200000</soft_erp>
+                <kp>100000.000000</kp>
+                <kd>1.000000</kd>
+                <max_vel>100.000000</max_vel>
+                <min_depth>0.001000</min_depth>
+              </ode>
+            </contact>
+          </surface>-->
         </collision>
         <visual >
@@ -54,13 +91,8 @@
 <inertial>
          <mass value = "0.05"/>
-<inertia ixx="0.000018" ixy ="0" ixz="0" iyy="0.00000722" iyz="0.0" izz="0.00000722"/>
-</inertial>
-<gazebo>
-<gravity> 1 </gravity>
-<dampingFactor>0.4</dampingFactor>
-<mu1>0.4</mu1>
-<mu2>0.4</mu2>
-<selfCollide>1</selfCollide>
-</gazebo>
+<inertia ixx="0.000847" ixy ="0" ixz="0" iyy="0.000847" iyz="0.0" izz="0.000847"/>
+</inertial>
+<gravity> 1 </gravity>
+<selfCollide>0</selfCollide>
       </link>
     <joint name="1${pos}" type="continuous">
@@ -69,8 +101,8 @@
      <origin xyz="${0.222*(-(0)*sin(yaw)+((0.05-0.28)*sin(pit)+(0.137)*cos(pit))*cos(yaw))} ${0.222*(((0)*cos(yaw))+((0.05-0.28)*sin(pit)+(0.137)*cos(pit))*sin(yaw))} ${0.222*((0.05-0.28)*cos(pit)+0.28-(0.137)*sin(pit)-0.28)}" rpy="${roll} ${pit} ${yaw}"/>
      <axis xyz="0 1 0">
-       <dynamics>
-        <damping>0.7</damping>
-        <friction>0.4</friction>
-       </dynamics>
+       <!--<dynamics>
+        <damping>0.7</damping>
+        <friction>0.4</friction>
+       </dynamics>-->
      </axis>
     </joint>
@@ -81,8 +113,29 @@
             <mesh filename="package://omni_bot/src/Wheel2_wheel_rightOrient.stl" scale=".0021 .0021 .0021"/>
           </geometry>
-          <friction>
-            <mu>0.4</mu>
-            <mu2>0.4</mu2>
-          </friction>
+          <!--<surface>
+            <friction>
+              <ode>
+                <mu>1.5</mu>
+                <mu2>1.5</mu2>
+                <fdir1>0.000000 0.000000 0.000000</fdir1>
+                <slip1>0.000000</slip1>
+                <slip2>0.000000</slip2>
+              </ode>
+            </friction>
+            <bounce>
+              <restitution_coefficient>0.000000</restitution_coefficient>
+              <threshold>100000.000000</threshold>
+            </bounce>
+            <contact>
+              <ode>
+                <soft_cfm>0.000000</soft_cfm>
+                <soft_erp>0.200000</soft_erp>
+                <kp>100000.000000</kp>
+                <kd>1.000000</kd>
+                <max_vel>100.000000</max_vel>
+                <min_depth>0.001000</min_depth>
+              </ode>
+            </contact>
+          </surface>-->
         </collision>
         <visual >
@@ -94,13 +147,8 @@
 <inertial>
          <mass value = "0.05"/>
-<inertia ixx="0.000018" ixy ="0" ixz="0" iyy="0.00000722" iyz="0.0" izz="0.00000722"/>
-</inertial>
-<gazebo>
-<gravity> 1 </gravity>
-<dampingFactor>0.4</dampingFactor>
-<mu1>0.4</mu1>
-<mu2>0.4</mu2>
-<selfCollide>1</selfCollide>
-</gazebo>
+<inertia ixx="0.000847" ixy ="0" ixz="0" iyy="0.000847" iyz="0.0" izz="0.000847"/>
+</inertial>
+<gravity> 1 </gravity>
+<selfCollide>0</selfCollide>
       </link>
     <joint name="2${pos}" type="continuous">
@@ -109,8 +157,8 @@
      <origin xyz="${0.222*(-(0.21)*sin(yaw)+((0.208-0.28)*sin(pit)+(0.137)*cos(pit))*cos(yaw))} ${0.222*(((0.21)*cos(yaw))+((0.208-0.28)*sin(pit)+(0.137)*cos(pit))*sin(yaw))} ${0.222*((0.208-0.28)*cos(pit)+0.28-(0.137)*sin(pit)-0.28)}" rpy="${roll} ${pit} ${yaw}"/>
      <axis xyz="0 0.31 0.95">
-      <dynamics>
-        <damping>0.7</damping>
-        <friction>0.4</friction>
-       </dynamics>
+       <!--<dynamics>
+        <damping>0.7</damping>
+        <friction>0.4</friction>
+       </dynamics>-->
      </axis>
     </joint>
@@ -121,8 +169,29 @@
             <mesh filename="package://omni_bot/src/Wheel2_wheel_rightOrient.stl" scale=".0021 .0021 .0021"/>
           </geometry>
-          <friction>
-            <mu>0.4</mu>
-            <mu2>0.4</mu2>
-          </friction>
+         <!--<surface>
+            <friction>
+              <ode>
+                <mu>1.5</mu>
+                <mu2>1.5</mu2>
+                <fdir1>0.000000 0.000000 0.000000</fdir1>
+                <slip1>0.000000</slip1>
+                <slip2>0.000000</slip2>
+              </ode>
+            </friction>
+            <bounce>
+              <restitution_coefficient>0.000000</restitution_coefficient>
+              <threshold>100000.000000</threshold>
+            </bounce>
+            <contact>
+              <ode>
+                <soft_cfm>0.000000</soft_cfm>
+                <soft_erp>0.200000</soft_erp>
+                <kp>100000.000000</kp>
+                <kd>1.000000</kd>
+                <max_vel>100.000000</max_vel>
+                <min_depth>0.001000</min_depth>
+              </ode>
+            </contact>
+          </surface>-->
         </collision>
         <visual >
@@ -134,13 +203,8 @@
 <inertial>
          <mass value = "0.05"/>
-<inertia ixx="0.000018" ixy ="0" ixz="0" iyy="0.00000722" iyz="0.0" izz="0.00000722"/>
-</inertial>
-<gazebo>
-<gravity> 1 </gravity>
-<dampingFactor>0.4</dampingFactor>
-<mu1>0.4</mu1>
-<mu2>0.4</mu2>
-<selfCollide>1</selfCollide>
-</gazebo>
+<inertia ixx="0.000847" ixy ="0" ixz="0" iyy="0.000847" iyz="0.0" izz="0.000847"/>
+</inertial>
+<gravity> 1 </gravity>
+<selfCollide>0</selfCollide>
       </link>
     <joint name="3${pos}" type="continuous">
@@ -149,8 +213,8 @@
      <origin xyz="${0.222*(-(0.14)*sin(yaw)+((0.47-0.28)*sin(pit)+(0.137)*cos(pit))*cos(yaw))} ${0.222*(((0.14)*cos(yaw))+((0.47-0.28)*sin(pit)+(0.137)*cos(pit))*sin(yaw))} ${0.222*((0.47-0.28)*cos(pit)+0.28-(0.137)*sin(pit)-0.28)}" rpy="${roll} ${pit} ${yaw}"/>
      <axis xyz="0 -0.81 0.59">
-      <dynamics>
-        <damping>0.7</damping>
-        <friction>0.4</friction>
-       </dynamics>
+      <!--<dynamics>
+        <damping>0.7</damping>
+        <friction>0.4</friction>
+       </dynamics>-->
      </axis>
     </joint>
@@ -161,8 +225,29 @@
             <mesh filename="package://omni_bot/src/Wheel2_wheel_rightOrient.stl" scale=".0021 .0021 .0021"/>
           </geometry>
-          <friction>
-            <mu>0.4</mu>
-            <mu2>0.4</mu2>
-          </friction>
+          <!--<surface>
+            <friction>
+              <ode>
+                <mu>1.5</mu>
+                <mu2>1.5</mu2>
+                <fdir1>0.000000 0.000000 0.000000</fdir1>
+                <slip1>0.000000</slip1>
+                <slip2>0.000000</slip2>
+              </ode>
+            </friction>
+            <bounce>
+              <restitution_coefficient>0.000000</restitution_coefficient>
+              <threshold>100000.000000</threshold>
+            </bounce>
+            <contact>
+              <ode>
+                <soft_cfm>0.000000</soft_cfm>
+                <soft_erp>0.200000</soft_erp>
+                <kp>100000.000000</kp>
+                <kd>1.000000</kd>
+                <max_vel>100.000000</max_vel>
+                <min_depth>0.001000</min_depth>
+              </ode>
+            </contact>
+          </surface>-->
         </collision>
         <visual >
@@ -174,13 +259,8 @@
 <inertial>
          <mass value = "0.05"/>
-<inertia ixx="0.000018" ixy ="0" ixz="0" iyy="0.00000722" iyz="0.0" izz="0.00000722"/>
-</inertial>
-<gazebo>
-<gravity> 1 </gravity>
-<dampingFactor>0.4</dampingFactor>
-<mu1>0.4</mu1>
-<mu2>0.4</mu2>
-<selfCollide>1</selfCollide>
-</gazebo>
+<inertia ixx="0.000847" ixy ="0" ixz="0" iyy="0.000847" iyz="0.0" izz="0.000847"/>
+</inertial>
+<gravity> 1 </gravity>
+<selfCollide>0</selfCollide>
       </link>
     <joint name="4${pos}" type="continuous">
@@ -189,8 +269,8 @@
      <origin xyz="${0.222*(-(-0.14)*sin(yaw)+((0.47-0.28)*sin(pit)+(0.137)*cos(pit))*cos(yaw))} ${0.222*(((-0.14)*cos(yaw))+((0.47-0.28)*sin(pit)+(0.137)*cos(pit))*sin(yaw))} ${0.222*((0.47-0.28)*cos(pit)+0.28-(0.137)*sin(pit)-0.28)}" rpy="${roll} ${pit} ${yaw}"/>
      <axis xyz="0 -0.81 -0.59">
-      <dynamics>
-        <damping>0.7</damping>
-        <friction>0.4</friction>
-       </dynamics>
+      <!--<dynamics>
+        <damping>0.7</damping>
+        <friction>0.4</friction>
+       </dynamics>-->
      </axis>
     </joint>
@@ -201,8 +281,29 @@
             <mesh filename="package://omni_bot/src/Wheel2_wheel_rightOrient.stl" scale=".0021 .0021 .0021"/>
           </geometry>
-          <friction>
-            <mu>0.4</mu>
-            <mu2>0.4</mu2>
-          </friction>
+          <!--<surface>
+            <friction>
+              <ode>
+                <mu>1.5</mu>
+                <mu2>1.5</mu2>
+                <fdir1>0.000000 0.000000 0.000000</fdir1>
+                <slip1>0.000000</slip1>
+                <slip2>0.000000</slip2>
+              </ode>
+            </friction>
+            <bounce>
+              <restitution_coefficient>0.000000</restitution_coefficient>
+              <threshold>100000.000000</threshold>
+            </bounce>
+            <contact>
+              <ode>
+                <soft_cfm>0.000000</soft_cfm>
+                <soft_erp>0.200000</soft_erp>
+                <kp>100000.000000</kp>
+                <kd>1.000000</kd>
+                <max_vel>100.000000</max_vel>
+                <min_depth>0.001000</min_depth>
+              </ode>
+            </contact>
+          </surface>-->
         </collision>
         <visual >
@@ -214,13 +315,8 @@
 <inertial>
          <mass value = "0.05"/>
-<inertia ixx="0.000018" ixy ="0" ixz="0" iyy="0.00000722" iyz="0.0" izz="0.00000722"/>
-</inertial>
-<gazebo>
-<gravity> 1 </gravity>
-<dampingFactor>0.4</dampingFactor>
-<mu1>0.4</mu1>
-<mu2>0.4</mu2>
-<selfCollide>1</selfCollide>
-</gazebo>
+<inertia ixx="0.000847" ixy ="0" ixz="0" iyy="0.000847" iyz="0.0" izz="0.000847"/>
+</inertial>
+<gravity> 1 </gravity>
+<selfCollide>0</selfCollide>
       </link>
     <joint name="5${pos}" type="continuous">
@@ -229,8 +325,8 @@
      <origin xyz="${0.222*(-(-0.22)*sin(yaw)+((0.21-0.28)*sin(pit)+(0.137)*cos(pit))*cos(yaw))} ${0.222*(((-0.22)*cos(yaw))+((0.21-0.28)*sin(pit)+(0.137)*cos(pit))*sin(yaw))} ${0.222*((0.21-0.28)*cos(pit)+0.28-(0.137)*sin(pit)-0.28)}" rpy="${roll} ${pit} ${yaw}"/>
      <axis xyz="0 0.31 -0.95">
-      <dynamics>
-        <damping>0.7</damping>
-        <friction>0.4</friction>
-       </dynamics>
+       <!--<dynamics>
+        <damping>0.7</damping>
+        <friction>0.4</friction>
+       </dynamics>-->
      </axis>
     </joint>
@@ -241,8 +337,29 @@
             <mesh filename="package://omni_bot/src/Wheel2_wheel_rightOrient.stl" scale=".0021 .0021 .0021"/>
           </geometry>
-          <friction>
-            <mu>0.4</mu>
-            <mu2>0.4</mu2>
-          </friction>
+          <!--<surface>
+            <friction>
+              <ode>
+                <mu>1.5</mu>
+                <mu2>1.5</mu2>
+                <fdir1>0.000000 0.000000 0.000000</fdir1>
+                <slip1>0.000000</slip1>
+                <slip2>0.000000</slip2>
+              </ode>
+            </friction>
+            <bounce>
+              <restitution_coefficient>0.000000</restitution_coefficient>
+              <threshold>100000.000000</threshold>
+            </bounce>
+            <contact>
+              <ode>
+                <soft_cfm>0.000000</soft_cfm>
+                <soft_erp>0.200000</soft_erp>
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