Commit message: Add files via upload

File: omni_bot/src/bot.xacro (robot description, xacro)
@@ -4,734 +4,557 @@
          xmlns:interface="http://ros.org/wiki/xacro"
          xmlns:sensor="http://playerstage.sourceforge.net/gazebo/xmlschema/#sensor" name="ballbot">
-   <xacro:macro name="omni" params="x y z roll pit yaw pos">
-      <link name="wheel${pos}">
-      <collision>
-         <origin xyz="0 0 0" rpy="${roll} ${pit} ${yaw}"/>
-          <geometry>
-            <mesh filename="package://omni_bot/src/Wheel2_Double_ohneRaeder.stl" scale=".0021 .0021 .0021"/>
-          </geometry>
-          <!--<surface>
-            <friction>
-              <ode>
-                <mu>1.5</mu>
-                <mu2>1.5</mu2>
-                <fdir1>0.000000 0.000000 0.000000</fdir1>
-                <slip1>0.000000</slip1>
-                <slip2>0.000000</slip2>
-              </ode>
-            </friction>
-            <bounce>
-              <restitution_coefficient>0.000000</restitution_coefficient>
-              <threshold>100000.000000</threshold>
-            </bounce>
-            <contact>
-              <ode>
-                <soft_cfm>0.000000</soft_cfm>
-                <soft_erp>0.200000</soft_erp>
-                <kp>100000.000000</kp>
-                <kd>1.000000</kd>
-                <max_vel>100.000000</max_vel>
-                <min_depth>0.001000</min_depth>
-              </ode>
-            </contact>
-          </surface>-->
-         </collision>
-      <visual>
-         <origin xyz="0 0 0" rpy="${roll} ${pit} ${yaw}"/>
-          <geometry>
-            <mesh filename="package://omni_bot/src/Wheel2_Double_ohneRaeder.stl" scale=".0021 .0021 .0021"/>
-          </geometry>
-         </visual>
-       <inertial>
-          <origin xyz="0 0 0" rpy="${roll} ${pit} ${yaw}"/>
-         <mass value = "0.55"/>
-    <inertia ixx="0.0005" ixy ="0" ixz="0" iyy="0.0005" iyz="0" izz="0.001"/>
-    </inertial>
-      <gravity> 1 </gravity>
-      <selfCollide>0</selfCollide>
-      </link>
-     <link name="roller1${pos}">
-       <collision >
-           <origin xyz="0 0 0" rpy="0 0 1.57079"/>
-          <geometry>
-            <mesh filename="package://omni_bot/src/Wheel2_wheel_rightOrient.stl" scale=".0021 .0021 .0021"/>
-          </geometry>
-          <!--<surface>
-            <friction>
-              <ode>
-                <mu>1.5</mu>
-                <mu2>1.5</mu2>
-                <fdir1>0.000000 0.000000 0.000000</fdir1>
-                <slip1>0.000000</slip1>
-                <slip2>0.000000</slip2>
-              </ode>
-            </friction>
-            <bounce>
-              <restitution_coefficient>0.000000</restitution_coefficient>
-              <threshold>100000.000000</threshold>
-            </bounce>
-            <contact>
-              <ode>
-                <soft_cfm>0.000000</soft_cfm>
-                <soft_erp>0.200000</soft_erp>
-                <kp>100000.000000</kp>
-                <kd>1.000000</kd>
-                <max_vel>100.000000</max_vel>
-                <min_depth>0.001000</min_depth>
-              </ode>
-            </contact>
-          </surface>-->
-        </collision>
-        <visual >
-           <origin xyz="0 0 0" rpy="0 0 1.57079"/>
-           <geometry>
-            <mesh filename="package://omni_bot/src/Wheel2_wheel_rightOrient.stl" scale=".0021 .0021 .0021"/>
-          </geometry>
-        </visual>
-<inertial>
-         <mass value = "0.05"/>
-<inertia ixx="0.000847" ixy ="0" ixz="0" iyy="0.000847" iyz="0.0" izz="0.000847"/>
-</inertial>
+<link name="dummy">
+   </link>
+ <xacro:macro name="omni" params="x y z roll pit yaw pos">
+  <link name="wheel${pos}">
+    <collision>
+    <origin xyz="0 0 0" rpy="${roll} ${pit} ${yaw}"/>
+      <geometry>
+        <mesh filename="package://omni_bot/src/Wheel2_Double_ohneRaeder.stl" scale=".0021 .0021 .0021"/>
+      </geometry>
+      <surface>
+        <friction>
+          <ode>
+            <mu>100000.0</mu>
+            <mu2>100000.0</mu2>
+          </ode>
+        </friction>
+      </surface>
+    </collision>
+    <visual>
+    <origin xyz="0 0 0" rpy="${roll} ${pit} ${yaw}"/>
+      <geometry>
+        <mesh filename="package://omni_bot/src/Wheel2_Double_ohneRaeder.stl" scale=".0021 .0021 .0021"/>
+      </geometry>
+    </visual>
+    <inertial>
+      <origin xyz="0 0 0" rpy="${roll} ${pit} ${yaw}"/>
+      <mass value = "2.5"/>
+      <inertia ixx="0.00508333333333" ixy="0" ixz="0" iyy="0.00508333333333" iyz="0" izz="0.005"/>
+    </inertial>
+    <!-- <gravity> 1 </gravity>
+    <selfCollide>0</selfCollide> -->
+  </link>
+  <link name="roller1${pos}">
+    <collision >
+      <origin xyz="0 0 0" rpy="0 0 1.57079"/>
+      <geometry>
+        <mesh filename="package://omni_bot/src/Wheel2_wheel_rightOrient.stl" scale=".0021 .0021 .0021"/>
+      </geometry>
+      <surface>
+        <friction>
+          <ode>
+            <mu>100000.0</mu>
+            <mu2>100000.0</mu2>
+          </ode>
+        </friction>
+      </surface>
+    </collision>
+    <visual >
+      <origin xyz="0 0 0" rpy="0 0 1.57079"/>
+      <geometry>
+        <mesh filename="package://omni_bot/src/Wheel2_wheel_rightOrient.stl" scale=".0021 .0021 .0021"/>
+      </geometry>
+    </visual>
+    <inertial>
+      <origin xyz="0 0 0" rpy="0 0 1.57079"/>
+      <mass value = "0.1"/>
+      <inertia ixx="0.0000847" ixy ="0" ixz="0" iyy="0.0000847" iyz="0.0" izz="0.0000847"/>
+    </inertial>
+<!-- <gravity> 1 </gravity>
+<selfCollide>0</selfCollide> -->
+  </link>
+  <joint name="1${pos}" type="continuous">
+    <parent link="wheel${pos}"/>
+    <child link="roller1${pos}"/>
+    <origin xyz="${0.222*(-(0)*sin(yaw)+((0.05-0.28)*sin(pit)+(0.137)*cos(pit))*cos(yaw))} ${0.222*(((0)*cos(yaw))+((0.05-0.28)*sin(pit)+(0.137)*cos(pit))*sin(yaw))} ${0.222*((0.05-0.28)*cos(pit)+0.28-(0.137)*sin(pit)-0.28)}" rpy="${roll} ${pit} ${yaw}"/>
+    <axis xyz="0 1 0"/>
+    <limit effort="1.5" velocity="100"/>
+       <!-- <dynamics>
+        <damping>0.7</damping>
+        <friction>0.4</friction>
+       </dynamics> -->
+  </joint>
+  <link name="roller2${pos}">
+    <collision >
+      <origin xyz="0 0 0" rpy="0 -1.25664 1.57079"/>
+      <geometry>
+        <mesh filename="package://omni_bot/src/Wheel2_wheel_rightOrient.stl" scale=".0021 .0021 .0021"/>
+      </geometry>
+      <surface>
+        <friction>
+          <ode>
+            <mu>100000.0</mu>
+            <mu2>100000.0</mu2>
+          </ode>
+        </friction>
+      </surface>
+    </collision>
+    <visual >
+      <origin xyz="0 0 0" rpy="0 -1.25664 1.57079"/>
+      <geometry>
+        <mesh filename="package://omni_bot/src/Wheel2_wheel_rightOrient.stl" scale=".0021 .0021 .0021"/>
+      </geometry>
+    </visual>
+    <inertial>
+      <origin xyz="0 0 0" rpy="0 -1.25664 1.57079"/>
+      <mass value = "0.1"/>
+      <inertia ixx="0.0000847" ixy ="0" ixz="0" iyy="0.0000847" iyz="0.0" izz="0.0000847"/>
+    </inertial>
+<!--
 <gravity> 1 </gravity>
 <selfCollide>0</selfCollide>
-      </link>
-    <joint name="1${pos}" type="continuous">
-     <parent link="wheel${pos}"/>
-     <child link="roller1${pos}"/>
-     <origin xyz="${0.222*(-(0)*sin(yaw)+((0.05-0.28)*sin(pit)+(0.137)*cos(pit))*cos(yaw))} ${0.222*(((0)*cos(yaw))+((0.05-0.28)*sin(pit)+(0.137)*cos(pit))*sin(yaw))} ${0.222*((0.05-0.28)*cos(pit)+0.28-(0.137)*sin(pit)-0.28)}" rpy="${roll} ${pit} ${yaw}"/>
-     <axis xyz="0 1 0">
-       <!--<dynamics>
-        <damping>0.7</damping>
-        <friction>0.4</friction>
-       </dynamics>-->
-     </axis>
-    </joint>
-    <link name="roller2${pos}">
-       <collision >
-           <origin xyz="0 0 0" rpy="0 -1.25664 1.57079"/>
-          <geometry>
-            <mesh filename="package://omni_bot/src/Wheel2_wheel_rightOrient.stl" scale=".0021 .0021 .0021"/>
-          </geometry>
-          <!--<surface>
-            <friction>
-              <ode>
-                <mu>1.5</mu>
-                <mu2>1.5</mu2>
-                <fdir1>0.000000 0.000000 0.000000</fdir1>
-                <slip1>0.000000</slip1>
-                <slip2>0.000000</slip2>
-              </ode>
-            </friction>
-            <bounce>
-              <restitution_coefficient>0.000000</restitution_coefficient>
-              <threshold>100000.000000</threshold>
-            </bounce>
-            <contact>
-              <ode>
-                <soft_cfm>0.000000</soft_cfm>
-                <soft_erp>0.200000</soft_erp>
-                <kp>100000.000000</kp>
-                <kd>1.000000</kd>
-                <max_vel>100.000000</max_vel>
-                <min_depth>0.001000</min_depth>
-              </ode>
-            </contact>
-          </surface>-->
-        </collision>
-        <visual >
-           <origin xyz="0 0 0" rpy="0 -1.25664 1.57079"/>
-           <geometry>
-            <mesh filename="package://omni_bot/src/Wheel2_wheel_rightOrient.stl" scale=".0021 .0021 .0021"/>
-          </geometry>
-        </visual>
-<inertial>
-         <mass value = "0.05"/>
-<inertia ixx="0.000847" ixy ="0" ixz="0" iyy="0.000847" iyz="0.0" izz="0.000847"/>
-</inertial>
+ -->
+  </link>
+  <joint name="2${pos}" type="continuous">
+    <parent link="wheel${pos}"/>
+    <child link="roller2${pos}"/>
+    <origin xyz="${0.222*(-(0.21)*sin(yaw)+((0.208-0.28)*sin(pit)+(0.137)*cos(pit))*cos(yaw))} ${0.222*(((0.21)*cos(yaw))+((0.208-0.28)*sin(pit)+(0.137)*cos(pit))*sin(yaw))} ${0.222*((0.208-0.28)*cos(pit)+0.28-(0.137)*sin(pit)-0.28)}" rpy="${roll} ${pit} ${yaw}"/>
+    <axis xyz="0 0.31 0.95"/>
+    <limit effort="1.5" velocity="100"/>
+    <!-- <dynamics>
+        <damping>0.7</damping>
+        <friction>0.4</friction>
+       </dynamics> -->
+  </joint>
+  <link name="roller3${pos}">
+    <collision >
+      <origin xyz="0 0 0" rpy="0 -2.5132 1.57079"/>
+      <geometry>
+        <mesh filename="package://omni_bot/src/Wheel2_wheel_rightOrient.stl" scale=".0021 .0021 .0021"/>
+      </geometry>
+      <surface>
+        <friction>
+          <ode>
+            <mu>100000.0</mu>
+            <mu2>100000.0</mu2>
+          </ode>
+        </friction>
+      </surface>
+    </collision>
+    <visual >
+      <origin xyz="0 0 0" rpy="0 -2.5132 1.57079"/>
+      <geometry>
+        <mesh filename="package://omni_bot/src/Wheel2_wheel_rightOrient.stl" scale=".0021 .0021 .0021"/>
+      </geometry>
+    </visual>
+    <inertial>
+      <origin xyz="0 0 0" rpy="0 -2.5132 1.57079"/>
+      <mass value = "0.1"/>
+      <inertia ixx="0.0000847" ixy ="0" ixz="0" iyy="0.0000847" iyz="0.0" izz="0.0000847"/>
+    </inertial>
+<!--
 <gravity> 1 </gravity>
 <selfCollide>0</selfCollide>
-      </link>
-    <joint name="2${pos}" type="continuous">
-     <parent link="wheel${pos}"/>
-     <child link="roller2${pos}"/>
-     <origin xyz="${0.222*(-(0.21)*sin(yaw)+((0.208-0.28)*sin(pit)+(0.137)*cos(pit))*cos(yaw))} ${0.222*(((0.21)*cos(yaw))+((0.208-0.28)*sin(pit)+(0.137)*cos(pit))*sin(yaw))} ${0.222*((0.208-0.28)*cos(pit)+0.28-(0.137)*sin(pit)-0.28)}" rpy="${roll} ${pit} ${yaw}"/>
-     <axis xyz="0 0.31 0.95">
-       <!--<dynamics>
-        <damping>0.7</damping>
-        <friction>0.4</friction>
-       </dynamics>-->
-     </axis>
-    </joint>
-     <link name="roller3${pos}">
-        <collision >
-           <origin xyz="0 0 0" rpy="0 -2.5132 1.57079"/>
-          <geometry>
-            <mesh filename="package://omni_bot/src/Wheel2_wheel_rightOrient.stl" scale=".0021 .0021 .0021"/>
-          </geometry>
-         <!--<surface>
-            <friction>
-              <ode>
-                <mu>1.5</mu>
-                <mu2>1.5</mu2>
-                <fdir1>0.000000 0.000000 0.000000</fdir1>
-                <slip1>0.000000</slip1>
-                <slip2>0.000000</slip2>
-              </ode>
-            </friction>
-            <bounce>
-              <restitution_coefficient>0.000000</restitution_coefficient>
-              <threshold>100000.000000</threshold>
-            </bounce>
-            <contact>
-              <ode>
-                <soft_cfm>0.000000</soft_cfm>
-                <soft_erp>0.200000</soft_erp>
-                <kp>100000.000000</kp>
-                <kd>1.000000</kd>
-                <max_vel>100.000000</max_vel>
-                <min_depth>0.001000</min_depth>
-              </ode>
-            </contact>
-          </surface>-->
-        </collision>
-        <visual >
-           <origin xyz="0 0 0" rpy="0 -2.5132 1.57079"/>
-           <geometry>
-            <mesh filename="package://omni_bot/src/Wheel2_wheel_rightOrient.stl" scale=".0021 .0021 .0021"/>
-          </geometry>
-        </visual>
-<inertial>
-         <mass value = "0.05"/>
-<inertia ixx="0.000847" ixy ="0" ixz="0" iyy="0.000847" iyz="0.0" izz="0.000847"/>
-</inertial>
+ -->
+  </link>
+  <joint name="3${pos}" type="continuous">
+    <parent link="wheel${pos}"/>
+    <child link="roller3${pos}"/>
+    <origin xyz="${0.222*(-(0.14)*sin(yaw)+((0.47-0.28)*sin(pit)+(0.137)*cos(pit))*cos(yaw))} ${0.222*(((0.14)*cos(yaw))+((0.47-0.28)*sin(pit)+(0.137)*cos(pit))*sin(yaw))} ${0.222*((0.47-0.28)*cos(pit)+0.28-(0.137)*sin(pit)-0.28)}" rpy="${roll} ${pit} ${yaw}"/>
+    <axis xyz="0 -0.81 0.59"/>
+    <limit effort="1.5" velocity="100"/>
+      <!-- <dynamics>
+        <damping>0.7</damping>
+        <friction>0.4</friction>
+       </dynamics> -->
+  </joint>
+  <link name="roller4${pos}">
+    <collision >
+      <origin xyz="0 0 0" rpy="0 -3.7699 1.57079"/>
+      <geometry>
+        <mesh filename="package://omni_bot/src/Wheel2_wheel_rightOrient.stl" scale=".0021 .0021 .0021"/>
+      </geometry>
+      <surface>
+        <friction>
+          <ode>
+            <mu>100000.0</mu>
+            <mu2>100000.0</mu2>
+          </ode>
+        </friction>
+      </surface>
+    </collision>
+    <visual >
+      <origin xyz="0 0 0" rpy="0 -3.7699 1.57079"/>
+      <geometry>
+        <mesh filename="package://omni_bot/src/Wheel2_wheel_rightOrient.stl" scale=".0021 .0021 .0021"/>
+      </geometry>
+    </visual>
+    <inertial>
+      <origin xyz="0 0 0" rpy="0 -3.7699 1.57079"/>
+      <mass value = "0.1"/>
+      <inertia ixx="0.0000847" ixy ="0" ixz="0" iyy="0.0000847" iyz="0.0" izz="0.0000847"/>
+    </inertial>
+<!--
 <gravity> 1 </gravity>
 <selfCollide>0</selfCollide>
-      </link>
-    <joint name="3${pos}" type="continuous">
-     <parent link="wheel${pos}"/>
-     <child link="roller3${pos}"/>
-     <origin xyz="${0.222*(-(0.14)*sin(yaw)+((0.47-0.28)*sin(pit)+(0.137)*cos(pit))*cos(yaw))} ${0.222*(((0.14)*cos(yaw))+((0.47-0.28)*sin(pit)+(0.137)*cos(pit))*sin(yaw))} ${0.222*((0.47-0.28)*cos(pit)+0.28-(0.137)*sin(pit)-0.28)}" rpy="${roll} ${pit} ${yaw}"/>
-     <axis xyz="0 -0.81 0.59">
-      <!--<dynamics>
-        <damping>0.7</damping>
-        <friction>0.4</friction>
-       </dynamics>-->
-     </axis>
-    </joint>
-     <link name="roller4${pos}">
-           <collision >
-           <origin xyz="0 0 0" rpy="0 -3.7699 1.57079"/>
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
Commit message: Add files via upload

File: omni_bot/src/bot.xacro (robot description, xacro)
@@ -562,6 +562,5 @@
    </plugin>
 </gazebo>
-<!--
-<link name="imu_link">
+<!-- <link name="imu_link">
   <inertial>
     <mass value="0.01"/>
@@ -587,9 +586,7 @@
     <parent link="body"/>
     <child link="imu_link"/>
-</joint>
--->
+</joint> -->
 <!-- Change imu topic name to bot specific to prevent clash   -->
-<!--
-<gazebo>
+<!-- <gazebo>
   <plugin name="imu_plugin" filename="libgazebo_ros_imu.so">
     <alwaysOn>true</alwaysOn>
@@ -602,5 +599,5 @@
     </plugin>
 </gazebo>
- -->
+  -->
 </robot>
 <!--
